File: electronics/single_face_controller_prototype/single_face_controller_prototype.kicad_sch (KiCad schematic)
At the start: 0 parts

Commit message: Add STSPIN32F0A mcu/bldc controller
Parts:
- added U?: STSPIN32F0A, symbol User:STSPIN32F0A
Connections:
- new net EPAD: U?.0 (EPAD), U?.44 (GND)
Changed lines of the file:
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@@
 (kicad_sch (version 20210126) (generator eeschema)
   (paper "A4")
-  (symbol_instances)
+  (symbol (lib_id "User:STSPIN32F0A") (at 127 101.6 0) (unit 1)
+    (in_bom yes) (on_board yes)
+    (property "Reference" "U?" (id 0) (at 127 59.8128 0))
+    (property "Value" "STSPIN32F0A" (id 1) (at 127 62.1115 0))
+    (property "Footprint" "" (id 2) (at 111.76 139.7 0)
+      (effects (font (size 1.27 1.27)) (justify right) hide)
+    )
+    (property "Datasheet" "https://www.st.com/resource/en/datasheet/stspin32f0a.pdf" (id 3) (at 165.1 99.06 0)
+      (effects (font (size 1.27 1.27)) hide)
+    )
+    (pin "0")
+    (pin "1")
+    (pin "10")
+    (pin "11")
+    (pin "12")
+    (pin "13")
+    (pin "14")
+    (pin "15")
+    (pin "16")
+    (pin "17")
+    (pin "18")
+    (pin "19")
+    (pin "2")
+    (pin "20")
+    (pin "21")
+    (pin "22")
+    (pin "23")
+    (pin "24")
+    (pin "25")
+    (pin "26")
+    (pin "27")
+    (pin "28")
+    (pin "29")
+    (pin "3")
+    (pin "30")
+    (pin "31")
+    (pin "32")
+    (pin "33")
+    (pin "34")
+    (pin "35")
+    (pin "36")
+    (pin "37")
+    (pin "38")
+    (pin "39")
+    (pin "4")
+    (pin "40")
+    (pin "41")
+    (pin "42")
+    (pin "43")
+    (pin "44")
+    (pin "45")
+    (pin "46")
+    (pin "47")
+    (pin "48")
+    (pin "5")
+    (pin "6")
+    (pin "7")
+    (pin "8")
+    (pin "9")
+  )
+  (sheet_instances
+    (path "/" (page "1"))
+  )
+  (symbol_instances
+    (path "/6b0556ca-7022-41ff-af7b-e2a327ac1698"
+      (reference "U?") (unit 1) (value "STSPIN32F0A") (footprint "")
+    )
+  )
 )
